File: project/hardware/matrix-game.kicad_pcb (KiCad board)
At the start: 2 copper layers, 100 x 100 mm, 32 parts, among them SW1 button_center, SW2 button_left, SW3 button_down, SW4 button_right, SW5 button_up, U1 NUCLEO-F042K6, U2 MAX7219, U3 SSD1306

Commit message: [project/hardware/layout] more layouting
Signed-off-by: Timon Burkard <timon.burkard@gwf.ch>
Connections:
- net Net-(U1-PF1/D8) renamed lcd_scl
Changed lines of the file:
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@@
 	(net 31 "Net-(U1-PA5{slash}A4)")
 	(net 32 "unconnected-(U1-PA6{slash}A5-PadCN4_7)")
-	(net 33 "Net-(U1-PF1{slash}D8)")
+	(net 33 "lcd_scl")
 	(net 34 "unconnected-(U1-PB3{slash}D13-PadCN4_15)")
 	(net 35 "unconnected-(U1-PA10{slash}D0-PadCN3_2)")
@@
 			(net 47 "unconnected-(U2-DOUT-Pad24)")
 			(pinfunction "DOUT")
-			(pintype "output")
+			(pintype "output+no_connect")
 		)
 		(model "${KICAD8_3DMODEL_DIR}/Package_DIP.3dshapes/DIP-24_W7.62mm_Socket.wrl"
@@
 			(layers "*.Cu" "*.Mask")
 			(remove_unused_layers no)
-			(net 33 "Net-(U1-PF1{slash}D8)")
+			(net 33 "lcd_scl")
 			(pinfunction "SCL")
 			(pintype "input")
@@
 			(net 45 "unconnected-(U1-PA9{slash}D1-PadCN3_1)")
 			(pinfunction "PA9/D1")
-			(pintype "bidirectional")
+			(pintype "bidirectional+no_connect")
 			(solder_mask_margin 0.102)
 		)
@@
 			(net 35 "unconnected-(U1-PA10{slash}D0-PadCN3_2)")
 			(pinfunction "PA10/D0")
-			(pintype "bidirectional")
+			(pintype "bidirectional+no_connect")
 			(solder_mask_margin 0.102)
 		)
@@
 			(net 39 "unconnected-(U1-~{RST}_CN3-PadCN3_3)")
 			(pinfunction "~{RST}_CN3")
-			(pintype "bidirectional")
+			(pintype "bidirectional+no_connect")
 			(solder_mask_margin 0.102)
 		)
@@
 			(net 36 "unconnected-(U1-PB7{slash}D4-PadCN3_7)")
 			(pinfunction "PB7/D4")
-			(pintype "bidirectional")
+			(pintype "bidirectional+no_connect")
 			(solder_mask_margin 0.102)
 		)
@@
 			(net 46 "unconnected-(U1-PB6{slash}D5-PadCN3_8)")
 			(pinfunction "PB6/D5")
-			(pintype "bidirectional")
+			(pintype "bidirectional+no_connect")
 			(solder_mask_margin 0.102)
 		)
@@
 			(net 29 "unconnected-(U1-PF0{slash}D7-PadCN3_10)")
 			(pinfunction "PF0/D7")
-			(pintype "bidirectional")
+			(pintype "bidirectional+no_connect")
 			(solder_mask_margin 0.102)
 		)
@@
 			(layers "*.Cu" "*.Mask")
 			(remove_unused_layers no)
-			(net 33 "Net-(U1-PF1{slash}D8)")
+			(net 33 "lcd_scl")
 			(pinfunction "PF1/D8")
 			(pintype "bidirectional")
@@
 			(net 43 "unconnected-(U1-PB4{slash}D12-PadCN3_15)")
 			(pinfunction "PB4/D12")
-			(pintype "bidirectional")
+			(pintype "bidirectional+no_connect")
 			(solder_mask_margin 0.102)
 		)
@@
 			(net 41 "unconnected-(U1-VIN-PadCN4_1)")
 			(pinfunction "VIN")
-			(pintype "power_in")
+			(pintype "power_in+no_connect")
 			(solder_mask_margin 0.102)
 		)
@@
 			(net 27 "unconnected-(U1-~{RST}_CN4-PadCN4_3)")
 			(pinfunction "~{RST}_CN4")
-			(pintype "bidirectional")
+			(pintype "bidirectional+no_connect")
 			(solder_mask_margin 0.102)
 		)
@@
 			(net 40 "unconnected-(U1-PA2{slash}A7-PadCN4_5)")
 			(pinfunction "PA2/A7")
-			(pintype "bidirectional")
+			(pintype "bidirectional+no_connect")
 			(solder_mask_margin 0.102)
 		)
@@
 			(net 32 "unconnected-(U1-PA6{slash}A5-PadCN4_7)")
 			(pinfunction "PA6/A5")
-			(pintype "bidirectional")
+			(pintype "bidirectional+no_connect")
 			(solder_mask_margin 0.102)
 		)
@@
 			(net 44 "unconnected-(U1-PA1{slash}A1-PadCN4_11)")
 			(pinfunction "PA1/A1")
-			(pintype "bidirectional")
+			(pintype "bidirectional+no_connect")
 			(solder_mask_margin 0.102)
 		)
@@
 			(net 26 "unconnected-(U1-PA0{slash}A0-PadCN4_12)")
 			(pinfunction "PA0/A0")
-			(pintype "bidirectional")
+			(pintype "bidirectional+no_connect")
 			(solder_mask_margin 0.102)
 		)
@@
 			(net 30 "unconnected-(U1-AREF-PadCN4_13)")
 			(pinfunction "AREF")
-			(pintype "input")
+			(pintype "input+no_connect")
 			(solder_mask_margin 0.102)
 		)
@@
 			(net 34 "unconnected-(U1-PB3{slash}D13-PadCN4_15)")
 			(pinfunction "PB3/D13")
-			(pintype "bidirectional")
+			(pintype "bidirectional+no_connect")
 			(solder_mask_margin 0.102)
 		)
